File: FTCMS_V2.2/alte platine/FTCMS_V2.2.kicad_pcb (KiCad board)
At the start: 2 copper layers, 95 x 64.9 mm, 113 parts, among them J1 Conn_01x20_Female, J2 Conn_02x10_Odd_Even, J3 ToSlave, J4 Conn_02x02_Odd_Even, J6 ToMaster, Q1 Q_NPN_BCE DZT5551, U1 ADBMS1818ASWAZ, U2 MAX9031AU

Commit message: platine debug 1
Parts:
- renumbered C27 to 24, C24 to C27
