File: FTCMS_V2.2/FTCMS_V2.2.kicad_sch (KiCad schematic)
At the start: 113 parts, among them J1 Conn_01x20_Female, J2 Conn_02x10_Odd_Even, J3 ToSlave, J4 ToMaster, J5 Conn_02x02_Odd_Even, Q1 Q_NPN_BCE DZT5551, U1 MAX9031AU, U2 ADBMS1818ASWAZ

Commit message: platine debug 1
Parts:
- renumbered C20 to C1, C9 to C11, C8 to C12, C7 to C13, C6 to C14, C5 to C15, C4 to C16, C3 to C17, C2 to C18, C1 to C19, C18 to C2, C28 to C20, C32 to C21, C26 to C24, C19 to C28, C31 to C29, C17 to C3, C29 to C31, C27 to C32, C16 to C4, C15 to C5, C14 to C6, C13 to C7, C12 to C8, C11 to C9, J4 to J6, JP4 to JP1, JP5 to JP2, JP8 to JP5, JP9 to JP6, JP6 to JP7, JP7 to JP8, R20 to R0, R19 to R1, R9 to R11, R8 to R12, R7 to R13, R6 to R14, R5 to R15, R4 to R16, R3 to R17, R2 to R18, R1 to R19, R18 to R2, R31 to R20, R30 to R22, R21 to R23, R22 to R25, R23 to R26, R17 to R3, R24 to R32, R16 to R4, R15 to R5, R14 to R6, R13 to R7, R12 to R8, R11 to R9, U2 to U1, U1 to U2

Commit message: FCTMS rebuild
Parts:
- removed JP1: SPI Mode, Jumper:SolderJumper-2_P1.3mm_Open_TrianglePad1.0x1.5mm, symbol Jumper:SolderJumper_2_Open
- removed JP2: isoSPI Mode, Jumper:SolderJumper-2_P1.3mm_Open_TrianglePad1.0x1.5mm, symbol Jumper:SolderJumper_2_Open
- added JP10: SPI - isoSPI, Jumper:SolderJumper-3_P2.0mm_Open_TrianglePad1.0x1.5mm, symbol Jumper:SolderJumper_3_Open
- J1, J2: footprint Project_Lib:Molex_Micro-Fit_3.0_43045-2000_2x10_P3.00mm_Horizontal -> Connector_PinSocket_2.54mm:PinSocket_2x10_P2.54mm_Vertical
- J3, J6: footprint Connector_Molex:Molex_Micro-Fit_3.0_43045-0212_2x01_P3.00mm_Vertical -> Connector_Molex:Molex_Micro-Fit_3.0_43650-0200_1x02_P3.00mm_Horizontal
- TR1: footprint MyFootprints:H0068ANL -> Audio_Module:H0068ANL
- renumbered C25 to C22, C22 to C25, C21 to C26, C24 to C27, JP2 to JP4, JP1 to JP9, R26 to R21, R29 to R24, R25 to R27, R27 to R30, R28 to R31
Connections:
- net GNDREF: now also JP10.1 (A)
- net ISOMD: now also JP10.2 (C)
- net Vreg: now also JP10.3 (B)

Commit message: 3d modelle der molex-stecker hinzugefügt
Connections:
- net GNDREF: now also U1.EPAD1 (V-)
- no-connect marks 6 -> 5
Other:
- moved on the sheet: R23
Changed lines of the file:
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@@
   (no_connect (at 175.895 258.445))
   (no_connect (at 54.61 89.535))
-  (no_connect (at 185.42 67.31))
   (no_connect (at 339.09 186.055))
   (no_connect (at 339.09 175.895))
@@
     (stroke (width 0) (type default))
   )
-  (wire (pts (xy 192.405 61.595) (xy 196.215 61.595))
+  (wire (pts (xy 193.04 60.96) (xy 199.39 60.96))
     (stroke (width 0) (type default))
   )
@@
     (stroke (width 0) (type default))
   )
-  (wire (pts (xy 185.42 72.39) (xy 192.405 72.39))
+  (wire (pts (xy 185.42 72.39) (xy 193.04 72.39))
     (stroke (width 0) (type default))
   )
@@
     (stroke (width 0) (type default))
   )
-  (wire (pts (xy 188.595 57.785) (xy 188.595 69.85))
+  (wire (pts (xy 191.77 57.15) (xy 191.77 69.85))
     (stroke (width 0) (type default))
   )
@@
     (stroke (width 0) (type default))
   )
-  (wire (pts (xy 192.405 72.39) (xy 192.405 61.595))
+  (wire (pts (xy 193.04 72.39) (xy 193.04 60.96))
     (stroke (width 0) (type default))
   )
@@
     (stroke (width 0) (type default))
   )
-  (wire (pts (xy 196.215 61.595) (xy 196.215 57.785))
+  (wire (pts (xy 199.39 60.96) (xy 199.39 57.15))
     (stroke (width 0) (type default))
   )
@@
     (stroke (width 0) (type default))
   )
-  (wire (pts (xy 188.595 69.85) (xy 185.42 69.85))
+  (wire (pts (xy 191.77 69.85) (xy 185.42 69.85))
     (stroke (width 0) (type default))
   )
@@
     )
   )
-  (global_label "IPB" (shape input) (at 188.595 57.785 180) (fields_autoplaced)
+  (global_label "IPB" (shape input) (at 191.77 57.15 180) (fields_autoplaced)
     (effects (font (size 1.27 1.27)) (justify right))
-    (property "Intersheetrefs" "${INTERSHEET_REFS}" (at 182.465 57.785 0)
+    (property "Intersheetrefs" "${INTERSHEET_REFS}" (at 185.64 57.15 0)
       (effects (font (size 1.27 1.27)) (justify right) hide)
     )
@@
     )
   )
-  (global_label "IMB" (shape input) (at 196.215 57.785 0) (fields_autoplaced)
-    (effects (font (size 1.27 1.27)) (justify left))
-    (property "Intersheetrefs" "${INTERSHEET_REFS}" (at 201.9543 57.7056 0)
+  (global_label "IMB" (shape input) (at 199.39 57.15 0) (fields_autoplaced)
+    (effects (font (size 1.27 1.27)) (justify left))
+    (property "Intersheetrefs" "${INTERSHEET_REFS}" (at 205.1293 57.0706 0)
       (effects (font (size 1.27 1.27)) (justify left) hide)
     )
@@
     )
   )
+  (global_label "V-" (shape input) (at 185.42 67.31 0) (fields_autoplaced)
+    (effects (font (size 1.27 1.27)) (justify left))
+    (property "Intersheetrefs" "${INTERSHEET_REFS}" (at 191.0662 67.31 0)
+      (effects (font (size 1.27 1.27)) (justify left) hide)
+    )
+  )
   (global_label "S2" (shape input) (at 139.7 153.67 0) (fields_autoplaced)
     (effects (font (size 1.27 1.27)) (justify left))
@@
     )
   )
-  (symbol (lib_id "Device:R") (at 192.405 57.785 90) (unit 1)
+  (symbol (lib_id "Device:R") (at 195.58 57.15 90) (unit 1)
     (in_bom yes) (on_board yes) (dnp no) (fields_autoplaced)
-    (property "Reference" "R23" (at 192.405 53.34 90)
-      (effects (font (size 1.27 1.27)))
-    )
-    (property "Value" "100/120R" (at 192.405 55.88 90)
-      (effects (font (size 1.27 1.27)))
-    )
-    (property "Footprint" "Resistor_SMD:R_1206_3216Metric_Pad1.30x1.75mm_HandSolder" (at 192.405 59.563 90)
-      (effects (font (size 1.27 1.27)) hide)
-    )
-    (property "Datasheet" "~" (at 192.405 57.785 0)
-      (effects (font (size 1.27 1.27)) hide)
-    )
+    (property "Reference" "R23" (at 195.58 52.705 90)
+      (effects (font (size 1.27 1.27)))
+    )
+    (property "Value" "100/120R" (at 195.58 55.245 90)
+      (effects (font (size 1.27 1.27)))
+    )
+    (property "Footprint" "Resistor_SMD:R_1206_3216Metric_Pad1.30x1.75mm_HandSolder" (at 195.58 58.928 90)
+      (effects (font (size 1.27 1.27)) hide)
+    )
+    (property "Datasheet" "~" (at 195.58 57.15 0)
+      (effects (font (size 1.27 1.27)) hide)
+    )
